File: switcher/switcher.sch (KiCad schematic (older format))
At the start: 7 parts

Commit message: update
Parts:
- removed C?: 0.1uF, symbol Device:C
- added C1, C2, C3: CP, Capacitor_THT:CP_Radial_D8.0mm_P3.80mm, symbol Device:CP
- added J1: ADA_TPL5100, Connector_PinSocket_2.54mm:PinSocket_1x05_P2.54mm_Vertical, symbol Connector:Conn_01x05_Female
- added J2: Screw_Terminal_01x02, TerminalBlock_4Ucon:TerminalBlock_4Ucon_1x02_P3.50mm_Vertical, symbol Connector:Screw_Terminal_01x02
- added J3: sreg, Connector_PinSocket_2.54mm:PinSocket_1x03_P2.54mm_Vertical, symbol Connector:Conn_01x03_Female
- added J4: Conn_01x05_Female, Connector_PinSocket_2.54mm:PinSocket_1x05_P2.54mm_Vertical, symbol Connector:Conn_01x05_Female
- added J5, J6: Conn_01x01_Female, Connector_PinSocket_2.54mm:PinSocket_1x01_P2.54mm_Vertical, symbol Connector:Conn_01x01_Female
- added R1: RD1, Resistor_THT:R_Axial_DIN0411_L9.9mm_D3.6mm_P7.62mm_Vertical, symbol Device:R
- added R2: RD2, Resistor_THT:R_Axial_DIN0411_L9.9mm_D3.6mm_P7.62mm_Vertical, symbol Device:R
- added R3: RD3, Resistor_THT:R_Axial_DIN0411_L9.9mm_D3.6mm_P7.62mm_Vertical, symbol Device:R
- added R4: RD4, Resistor_THT:R_Axial_DIN0411_L9.9mm_D3.6mm_P7.62mm_Vertical, symbol Device:R
- added SW1: SW_DIP_x04, Button_Switch_THT:SW_DIP_SPSTx04_Slide_6.7x11.72mm_W7.62mm_P2.54mm_LowProfile, symbol Switch:SW_DIP_x04
- D1: renamed from D?; footprint (none) -> Diode_THT:D_DO-41_SOD81_P10.16mm_Horizontal
- MMBT2N3904: footprint (none) -> Connector_PinSocket_2.54mm:PinSocket_1x03_P2.54mm_Vertical
- Q1, Q2: renamed from Q?; value Q_PMOS_GDS -> DMP2045U; footprint (none) -> Connector_PinSocket_2.54mm:PinSocket_1x03_P2.54mm_Vertical
- R5, R6: renamed from R?; footprint (none) -> Resistor_THT:R_Axial_DIN0411_L9.9mm_D3.6mm_P7.62mm_Vertical
Connections:
- net labels added: +3V3, +VDC, DONE, VDD-SWITCH
- net labels removed: GPIO3.3V, VDD
- wire segments 24 -> 86
Other:
- note added: "Switch Reg VX CUI 3V3"
