File: switcher/switcher.kicad_pcb (KiCad board)
At the start: 2 copper layers, 20 parts, among them J1 ADA_TPL5100, J2 Screw_Terminal_01x02, J3 sreg, J4 Conn_01x05_Female, J5 Conn_01x01_Female, J6 Conn_01x01_Female, Q1 DMP2045U, Q2 DMP2045U, SW1 SW_DIP_x04

Commit message: update
Other:
- board outline added: 90.2 x 57.2 mm
