File: switcher/switcher-smt.kicad_pcb (KiCad board)
At the start: 2 copper layers, 28 parts, among them J1 Screw_Terminal_01x02, J2 Screw_Terminal_01x02, J3 sreg, J4 Screw_Terminal_01x02, J5 Screw_Terminal_01x02, J6 Conn_01x06_Female, Q1 DMP2045U, Q2 DMP2045U, Q3 DMP2045U, Q4 DMP2045U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

Commit message: update
Parts:
- removed MH5: MountingHole, MountingHole:MountingHole_2.2mm_M2
- removed R7: RD5, Resistor_SMD:R_0603_1608Metric_Pad1.05x0.95mm_HandSolder
- added MH4: MountingHole, MountingHole:MountingHole_2.2mm_M2, F.Cu at (56.0, 44.9)
- added Q5: DMP2045U, Package_TO_SOT_SMD:SOT-23, F.Cu at (36.1, 24.6)
- added Q6: MMBT3904, Package_TO_SOT_SMD:SOT-23, F.Cu at (38.0, 28.7)
- added R10: 10K, Resistor_SMD:R_0603_1608Metric, F.Cu at (40.9, 28.7)
- added R11: 100K, Resistor_SMD:R_0603_1608Metric, F.Cu at (35.7, 31.6)
- added R5: RD5, Resistor_SMD:R_0603_1608Metric_Pad1.05x0.95mm_HandSolder, F.Cu at (37.5, 20.8)
- added R6: RD6, Resistor_SMD:R_0603_1608Metric_Pad1.05x0.95mm_HandSolder, F.Cu at (36.1, 20.8)
- added R9: 100K, Resistor_SMD:R_0603_1608Metric, F.Cu at (32.6, 31.5)
- J3: value sreg -> Conn_01x06_Female; footprint Connector_PinSocket_2.54mm:PinSocket_1x03_P2.54mm_Vertical -> Connector_PinSocket_2.54mm:PinSocket_1x06_P2.54mm_Vertical
- J6: value Conn_01x06_Female -> sreg; footprint Connector_PinSocket_2.54mm:PinSocket_1x06_P2.54mm_Vertical -> Connector_PinSocket_2.54mm:PinSocket_1x03_P2.54mm_Vertical
- Q3: value DMP2045U -> MMBT3904
- R8: value RD6 -> 10K; footprint Resistor_SMD:R_0603_1608Metric_Pad1.05x0.95mm_HandSolder -> Resistor_SMD:R_0603_1608Metric
- moved J5 36.0 mm to (53.0, 16.6), turned to 270 degrees
- moved J2 36.0 mm to (25.6, 38.3), turned to 90 degrees
- moved J6 30.3 mm to (27.5, 20.4), turned to 0 degrees
- moved J3 16.4 mm to (32.6, 43.1), turned to 90 degrees
- moved R8 13.6 mm to (32.6, 35.1)
- moved C2 13.5 mm to (33.3, 22.8)
- moved Q3 10.5 mm to (35.7, 35.1), turned to 270 degrees
- moved C4 8.68 mm to (35.2, 28.6), turned to 270 degrees
- moved D1 8.57 mm to (41.0, 37.1), turned to 90 degrees
- moved D2 7.25 mm to (32.9, 27.4), turned to 270 degrees
- moved C1 7.04 mm to (33.4, 19.2), turned to 270 degrees
- moved C3 6.66 mm to (38.6, 35.2), turned to 90 degrees
- moved U1 6.61 mm to (45.4, 31.6), turned to 90 degrees
- moved Q4 5.85 mm to (40.2, 24.6)
- moved Q2 5.63 mm to (37.5, 39.0), turned to 180 degrees
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Connections:
- C3 pad 1: VDD-SWITCH -> 3V3-SWITCH
- C4 pad 1: 3V3-SWITCH -> VDD-SWITCH
- D1 pad 1: VDD-SWITCH -> 3V3-SWITCH
- D2 pad 1: 3V3-SWITCH -> VDD-SWITCH
- J1 pad 1: DONE -> 3V3-SWITCH
- J2 pad 1: VDD-SWITCH -> +VDC
- J3 pad 1: +VDC -> VDD-SWITCH
- J3 pad 2: GND -> +VDC
- J3 pad 3: +3V3 -> GND
- J4 pad 1: 3V3-SWITCH -> DONE
- J5 pad 1: +VDC -> VDD-SWITCH
- J6 pad 3: VDD-SWITCH -> +3V3
- Q1 pad 1: SWITCHER -> Net-(Q1-Pad1)
- Q1 pad 2: +VDC -> +3V3
- Q2 pad 1: SWITCHER -> Net-(Q1-Pad1)
- Q2 pad 2: VDD-SWITCH -> 3V3-SWITCH
- Q3 pad 1: SWITCHER -> Net-(Q3-Pad1)
- Q3 pad 2: +3V3 -> GND
- Q3 pad 3: Net-(Q3-Pad3) -> Net-(Q1-Pad1)
- Q4 pad 1: SWITCHER -> Net-(Q4-Pad1)
- Q4 pad 2: 3V3-SWITCH -> +VDC
- Q4 pad 3: Net-(Q3-Pad3) -> Net-(Q4-Pad3)
- R8 pad 1: GND -> +3V3
- R8 pad 2: Net-(R8-Pad2) -> Net-(Q1-Pad1)
- SW1 pad 7: Net-(R8-Pad2) -> Net-(R6-Pad2)
Routing:
- net GND: track 0.00 -> 136.4 mm, vias 0 -> 4
- net VDD-SWITCH: track 0.00 -> 83.6 mm, vias 0 -> 2
- net +VDC: track 0.00 -> 74.3 mm, vias 0 -> 2
- net DELAY: track 0.00 -> 44.1 mm, vias 0 -> 2
- net +3V3: track 0.00 -> 37.7 mm, vias 0 -> 3
- net DONE: track 0.00 -> 27.4 mm, vias 0 -> 2
- net 3V3-SWITCH: track 0.00 -> 23.8 mm, vias 0 -> 1
- net SWITCHER: track 0.00 -> 17.7 mm, vias 0 -> 2
- net Net-(Q1-Pad1): track 0.00 -> 13.3 mm
- net Net-(Q4-Pad1): track 0.00 -> 12.7 mm
- net Net-(Q3-Pad1): track 0.00 -> 6.36 mm
- net Net-(Q4-Pad3): track 0.00 -> 6.34 mm
- net Net-(Q1-Pad3): track 0.00 -> 3.95 mm
- net Net-(R8-Pad2): track 2.88 -> 0.00 mm
- net Net-(R6-Pad2): track 0.00 -> 2.68 mm
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Other:
- board outline added: 39.7 x 40.3 mm
- net class power added: clearance 0.3, trace_width 0.4, via_dia 0.8, via_drill 0.4
- board text added: "(ver 0.1)"
- board text added: "10m"
- board text added: "10s"
- board text added: "1m"
- board text added: "30m"
- board text added: "3V3"
- board text added: "3VS"
- board text added: "60m"
- board text added: "DLY"
- board text added: "DN"
- board text added: "DONE"
- board text added: "GND"
- board text added: "VDC"
- board text added: "VIN"
- board text added: "VIN: 4.7-16V"
- board text added: "VINS"
- board text added: "edgecollective.io/"
- board text added: "timer-switch"
