File: switcher/switcher-smt.sch (KiCad schematic (older format))
At the start: 28 parts, among them J1 Screw_Terminal_01x02, J2 Screw_Terminal_01x02, J3 sreg, J4 Screw_Terminal_01x02, J5 Screw_Terminal_01x02, J6 Conn_01x06_Female, Q1 DMP2045U, Q2 DMP2045U, Q3 DMP2045U, Q4 DMP2045U, SW1 omron-a6h, U1 tpl5110

Commit message: update
Parts:
- added Q3, Q6: MMBT3904, Package_TO_SOT_SMD:SOT-23, symbol Transistor_BJT:MMBT3904
- added R10, R8: 10K, Resistor_SMD:R_0603_1608Metric, symbol Device:R
- added R11, R9: 100K, Resistor_SMD:R_0603_1608Metric, symbol Device:R
- gave numbers to parts that had none: 3
- renumbered C4 to C3, C3 to C4, D2 to D1, D1 to D2, J4 to J1, J5 to J2, J6 to J3, J1 to J4, J2 to J5, J3 to J6, MH5 to MH1, Q3 to Q1, Q4 to Q2, Q1 to Q4, Q2 to Q5, R7 to R5, R8 to R6
Connections:
- wire segments 69 -> 76
